File: Lotus 58 Classic/v1.28/Lotus58_Glow_128.kicad_pcb (KiCad board)
At the start: 2 copper layers, 139.1 x 107.7 mm, 122 parts, among them J1 PJ-320A, J2 Conn_01x02, P1 OLED, SW1 Kailh hotswap MX socket, SW10 Kailh hotswap MX socket, SW11 Kailh hotswap MX socket, SW12 Kailh hotswap MX socket, SW13 Kailh hotswap MX socket, SW14 Kailh hotswap MX socket, SW15 Kailh hotswap MX socket, SW16 Kailh hotswap MX socket, SW17 Kailh hotswap MX socket, SW18 Kailh hotswap MX socket, SW19 Kailh hotswap MX socket, SW2 Kailh hotswap MX socket, SW20 Kailh hotswap MX socket, SW21 Kailh hotswap MX socket, SW22 Kailh hotswap MX socket, SW23 Kailh hotswap MX socket, SW24 Kailh hotswap MX socket, SW25 Kailh hotswap MX socket, SW26 Kailh hotswap MX socket, SW27 Kailh hotswap MX socket, SW28 Kailh hotswap MX socket, SW29 Kailh hotswap MX socket, SW3 Kailh hotswap MX socket, SW30 Rotary_Encoder_Switch, SW31 Rotary_Encoder_Switch, SW4 Kailh hotswap MX socket, SW5 Kailh hotswap MX socket, SW6 Kailh hotswap MX socket, SW7 Kailh hotswap MX socket, SW8 Kailh hotswap MX socket, SW9 Kailh hotswap MX socket, U1 ProMicro, U2 SRV05-4

Commit message: Tweaked 1.41
Signed-off-by: TweetyDaBird <markus.knutsson@tweety.se>
Other:
- board text added: "DO NOT EVER USE SQUARE PIN_HEADERS!"
- board text added: "Power Switch"
- board text added: "RGB Switch"
- board text added: "TRRS NOT TO BE USED for wireless builds !!! To set switch as power switch or RGB selector close BOTH jumpers on the same side. Do NOT close jumpers on both sides !!!"
- board text removed: "Power"
- board text removed: "RGB"
- board text removed: "TRRS should NOT BE USED for wireless builds !!! Severe risk of damage !!! To set switch as power switch or RGB selector close BOTH jumpers on the same side."
Changed lines of the file:
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@@
   (title_block
     (title "Lotus 58 Glow")
-    (date "2023-12-27")
+    (date "2024-01-11")
     (rev "v1.28")
     (company "Markus Knutsson <markus.knutsson@tweety.se>")
@@
     (effects (font (size 0.75 0.75) (thickness 0.12)) (justify mirror))
   )
-  (gr_text "Place Encoder\non TOP of PCB." (at 91.43 58.91) (layer "B.SilkS")
+  (gr_text "Place Encoder\non TOP of PCB." (at 91.43 63.91) (layer "B.SilkS")
     (effects (font (size 0.75 0.75) (thickness 0.12)) (justify mirror))
   )
@@
     (effects (font (size 0.75 0.75) (thickness 0.12)) (justify left mirror))
   )
-  (gr_text "TRRS should NOT BE USED for wireless builds !!!\nSevere risk of damage !!!\n\nTo set switch as power switch or RGB selector \nclose BOTH jumpers on the same side." (at 102.89 91.55 90) (layer "B.SilkS")
+  (gr_text "TRRS NOT TO BE USED for wireless builds !!!\n\nTo set switch as power switch or RGB selector \nclose BOTH jumpers on the same side. \nDo NOT close jumpers on both sides !!!\n" (at 102.51 91.47 90) (layer "B.SilkS")
     (effects (font (size 0.75 0.75) (thickness 0.12)) (justify mirror))
   )
-  (gr_text "RGB" (at 99.9 39.02) (layer "B.SilkS")
-    (effects (font (size 0.75 0.75) (thickness 0.12)) (justify mirror))
+  (gr_text "RGB\nSwitch" (at 101.03 38.69) (layer "B.SilkS")
+    (effects (font (size 0.75 0.75) (thickness 0.12)) (justify left mirror))
   )
   (gr_text "- RST" (at 96.64 44.96 315) (layer "B.SilkS")
@@
     (effects (font (size 0.75 0.75) (thickness 0.12)) (justify mirror))
   )
+  (gr_text "DO NOT EVER\nUSE SQUARE\nPIN_HEADERS!" (at 91.57 58.34) (layer "B.SilkS")
+    (effects (font (size 0.75 0.75) (thickness 0.12)) (justify mirror))
+  )
   (gr_text "The controller MUST be placed in the correct orientation! Align it to match marked pins!\nThe controller sits with all components facing the keyboard PCB, and a flat backside towards the plate/case." (at 180.46 47.57 90) (layer "B.SilkS")
     (effects (font (size 0.75 0.75) (thickness 0.12)) (justify left mirror))
@@
     (effects (font (size 0.75 0.75) (thickness 0.12)) (justify left))
   )
-  (gr_text "Place Encoder\non TOP of PCB." (at 91.59 58.96) (layer "F.SilkS")
+  (gr_text "Place Encoder\non TOP of PCB." (at 91.59 63.96) (layer "F.SilkS")
     (effects (font (size 0.75 0.75) (thickness 0.12)))
   )
@@
     (effects (font (size 0.75 0.75) (thickness 0.12)))
   )
-  (gr_text "Power" (at 99.39 39.01) (layer "F.SilkS")
-    (effects (font (size 0.75 0.75) (thickness 0.12)))
+  (gr_text "Power\nSwitch" (at 97.34 38.69) (layer "F.SilkS")
+    (effects (font (size 0.75 0.75) (thickness 0.12)) (justify left))
   )
   (gr_text "- RST" (at 86.409492 45.74 -315) (layer "F.SilkS")
@@
     (effects (font (size 0.75 0.75) (thickness 0.12)))
   )
+  (gr_text "DO NOT EVER\nUSE SQUARE\nPIN_HEADERS!" (at 91.567 58.34) (layer "F.SilkS")
+    (effects (font (size 0.75 0.75) (thickness 0.12)))
+  )
