File: Lotus 58 USB-C/v1.41/Lotus58_Glow_141.kicad_pcb (KiCad board)
At the start: 2 copper layers, 139.1 x 107.7 mm, 119 parts, among them J3 USB_C_Receptacle_USB2.0, P1 OLED, SW1 Kailh hotswap MX socket, SW10 Kailh hotswap MX socket, SW11 Kailh hotswap MX socket, SW12 Kailh hotswap MX socket, SW13 Kailh hotswap MX socket, SW14 Kailh hotswap MX socket, SW15 Kailh hotswap MX socket, SW16 Kailh hotswap MX socket, SW17 Kailh hotswap MX socket, SW18 Kailh hotswap MX socket, SW19 Kailh hotswap MX socket, SW2 Kailh hotswap MX socket, SW20 Kailh hotswap MX socket, SW21 Kailh hotswap MX socket, SW22 Kailh hotswap MX socket, SW23 Kailh hotswap MX socket, SW24 Kailh hotswap MX socket, SW25 Kailh hotswap MX socket, SW26 Kailh hotswap MX socket, SW27 Kailh hotswap MX socket, SW28 Kailh hotswap MX socket, SW29 Kailh hotswap MX socket, SW3 Kailh hotswap MX socket, SW30 Rotary_Encoder_Switch, SW31 Rotary_Encoder_Switch, SW32 MSK12C02, SW33 MSK12C02, SW4 Kailh hotswap MX socket, SW5 Kailh hotswap MX socket, SW6 Kailh hotswap MX socket, SW7 Kailh hotswap MX socket, SW8 Kailh hotswap MX socket, SW9 Kailh hotswap MX socket, U1 ProMicro, U2 SRV05-4

Commit message: v1.41
Changed silkscreeen

Signed-off-by: TweetyDaBird <markus.knutsson@tweety.se>
Other:
- board text added: "LEFT HAND Solder jumpers on this side FIRST! DO NOT EVER USE SQUARE PIN-HEADERS! Controller is placed with components facing PCB. Encoder on TOP of PCB! Close for OLED on LEFT HAND"
- board text added: "RGB"
- board text added: "Use switch or ONE jumper"
- board text added: "locked"
- board text removed: "LEFT HAND Solder jumpers on this side FIRST! Place controller facing PCB. Encoder is placed on TOP of PCB! Close for OLED on LEFT HAND"
- board text removed: "RIGHT HAND Solder jumpers on this side FIRST! Place controller facing PCB. Encoder is placed on TOP of PCB! Close for OLED on RIGHT HAND"
Changed lines of the file:
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@@
     (property "ki_keywords" "usb universal serial bus type-C USB2.0")
     (attr smd)
-    (fp_text reference "J3" (at -6.858 -3.215 unlocked) (layer "F.SilkS")
+    (fp_text reference "J3" (at -6.858 -3.215 unlocked) (layer "F.SilkS") hide
         (effects (font (size 1 1) (thickness 0.15)))
     )
@@
     (fp_rect (start -3.28 1.06) (end 3.27 -1.07)
       (stroke (width 0.05) (type default)) (fill none) (layer "B.CrtYd"))
-    (pad "1" thru_hole circle (at -2.54 0 315) (size 1.397 1.397) (drill 0.8128) (layers "*.Cu" "*.Mask")
+    (pad "1" thru_hole circle (at -2.54 0 315) (size 1.5 1.5) (drill 0.8128) (layers "*.Cu" "*.Mask")
       (net 82 "EncB") (pintype "passive"))
-    (pad "2" thru_hole circle (at 2.54 0 315) (size 1.397 1.397) (drill 0.8128) (layers "*.Cu" "*.Mask")
+    (pad "2" thru_hole circle (at 2.54 0 315) (size 1.5 1.5) (drill 0.8128) (layers "*.Cu" "*.Mask")
       (net 34 "GND") (pintype "passive"))
     (model "discret/resistor.wrl"
@@
     (fp_rect (start -3.28 1.06) (end 3.27 -1.07)
       (stroke (width 0.05) (type default)) (fill none) (layer "B.CrtYd"))
-    (pad "1" thru_hole circle (at -2.54 0 135) (size 1.397 1.397) (drill 0.8128) (layers "*.Cu" "*.Mask")
+    (pad "1" thru_hole circle (at -2.54 0 135) (size 1.5 1.5) (drill 0.8128) (layers "*.Cu" "*.Mask")
       (net 34 "GND") (pintype "passive"))
-    (pad "2" thru_hole circle (at 2.54 0 135) (size 1.397 1.397) (drill 0.8128) (layers "*.Cu" "*.Mask")
+    (pad "2" thru_hole circle (at 2.54 0 135) (size 1.5 1.5) (drill 0.8128) (layers "*.Cu" "*.Mask")
       (net 83 "EncA") (pintype "passive"))
     (model "discret/resistor.wrl"
@@
     (effects (font (size 0.75 0.75) (thickness 0.12)) (justify left mirror))
   )
-  (gr_text "RIGHT HAND\nSolder jumpers\non this side\nFIRST!\n\n\n\nPlace\ncontroller\nfacing PCB.\n\n\n\nEncoder is\nplaced on\nTOP of PCB!\n\n\n\n\n\n\nClose for\nOLED \non RIGHT HAND" (at 91.567 55.65) (layer "B.SilkS")
+  (gr_text locked "RIGHT HAND\nSolder jumpers\non this side\nFIRST!\n\n\n\nDO NOT EVER\nUSE SQUARE\nPIN-HEADERS!\n\nController\nis placed\nwith \ncomponents\nfacing PCB.\n\n\nEncoder on\nTOP of PCB!\n\n\n\nClose for\nOLED on RIGHT HAND" (at 91.567 56.15375) (layer "B.SilkS")
     (effects (font (size 0.75 0.75) (thickness 0.12)) (justify mirror))
   )
@@
     (effects (font (size 0.75 0.75) (thickness 0.12)) (justify left mirror))
   )
-  (gr_text "Capacitors are\nonly used for\nthe encoder!" (at 103.59 58.73 90) (layer "B.SilkS")
+  (gr_text "Capacitors \nare only used \nfor the encoder!" (at 103.59 41.23 90) (layer "B.SilkS")
     (effects (font (size 0.75 0.75) (thickness 0.12)) (justify left mirror))
   )
@@
     (effects (font (size 1.2 1.2) (thickness 0.25)))
   )
+  (gr_text "Use switch\nor\nONE jumper\n" (at 104.29 47.34) (layer "F.SilkS")
+    (effects (font (size 0.75 0.75) (thickness 0.12)))
+  )
   (gr_text "3b. Solder the diodes to the COMPONENT SIDE of each hand. (Align stripe with square pad/arrow).\n3c. Solder RGB LED's as marked. Per-key RGB face UP & Glow RGB face DOWN!" (at 143.5 106.245 90) (layer "F.SilkS")
     (effects (font (size 0.75 0.75) (thickness 0.12)) (justify left))
   )
+  (gr_text "RGB" (at 102.11 40.5) (layer "F.SilkS")
+    (effects (font (size 0.75 0.75) (thickness 0.12)) (justify left))
+  )
   (gr_text "LEFT\nHAND" (at 97.455 75.25) (layer "F.SilkS")
     (effects (font (size 0.75 0.75) (thickness 0.12)) (justify left))
@@
     (effects (font (size 0.75 0.75) (thickness 0.12)) (justify left))
   )
-  (gr_text "LEFT HAND\nSolder jumpers\non this side\nFIRST!\n\n\n\nPlace\ncontroller\nfacing PCB.\n\n\n\nEncoder is\nplaced on\nTOP of PCB!\n\n\n\n\n\n\nClose for\nOLED \non LEFT HAND" (at 91.567 55.65) (layer "F.SilkS")
+  (gr_text "LEFT HAND\nSolder jumpers\non this side\nFIRST!\n\n\n\nDO NOT EVER\nUSE SQUARE\nPIN-HEADERS!\n\nController\nis placed\nwith \ncomponents\nfacing PCB.\n\n\nEncoder on\nTOP of PCB!\n\n\n\nClose for\nOLED on LEFT HAND" (at 91.567 56.15375) (layer "F.SilkS")
     (effects (font (size 0.75 0.75) (thickness 0.12)))
   )

Commit message: Tweaked 1.41
Signed-off-by: TweetyDaBird <markus.knutsson@tweety.se>
Other:
- board text added: "v1.4.1"
- board text removed: "v1.4.0"
Changed lines of the file:
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@@
   (title_block
     (title "Lotus 58 Glow")
-    (date "2023-11-21")
-    (rev "v1.4.0")
+    (date "2024-01-11")
+    (rev "v1.4.1")
     (company "Markus Knutsson <markus.knutsson@tweety.se>")
     (comment 1 "https://github.com/TweetyDaBird")
@@
     (effects (font (size 0.75 0.75) (thickness 0.12)) (justify mirror))
   )
-  (gr_text "v1.4.0" (at 88.85 110.79) (layer "B.SilkS")
+  (gr_text "v1.4.1" (at 88.85 110.79) (layer "B.SilkS")
     (effects (font (size 0.75 0.75) (thickness 0.12)) (justify mirror))
   )
@@
     (effects (font (size 0.75 0.75) (thickness 0.12)) (justify left))
   )
-  (gr_text "v1.4.0" (at 88.85 110.79) (layer "F.SilkS")
+  (gr_text "v1.4.1" (at 88.85 110.79) (layer "F.SilkS")
     (effects (font (size 0.75 0.75) (thickness 0.12)))
   )
