File: Lotus 58 Classic/v1.00/Lotus58_Classic.kicad_pcb (KiCad board)
At the start: 2 copper layers, 139.1 x 107.7 mm, 166 parts, among them J1 PJ-320A, P1 OLED, SW1 Kailh hotswap MX socket, SW10 Kailh hotswap MX socket, SW11 Kailh hotswap MX socket, SW12 Kailh hotswap MX socket, SW13 Kailh hotswap MX socket, SW14 Kailh hotswap MX socket, SW15 Kailh hotswap MX socket, SW16 Kailh hotswap MX socket, SW17 Kailh hotswap MX socket, SW18 Kailh hotswap MX socket, SW19 Kailh hotswap MX socket, SW2 Kailh hotswap MX socket, SW20 Kailh hotswap MX socket, SW21 Kailh hotswap MX socket, SW22 Kailh hotswap MX socket, SW23 Kailh hotswap MX socket, SW24 Kailh hotswap MX socket, SW25 Kailh hotswap MX socket, SW26 Kailh hotswap MX socket, SW27 Kailh hotswap MX socket, SW28 Kailh hotswap MX socket, SW29 Kailh hotswap MX socket, SW3 Kailh hotswap MX socket, SW30 Rotary_Encoder_Switch, SW31 Rotary_Encoder_Switch, SW4 Kailh hotswap MX socket, SW5 Kailh hotswap MX socket, SW6 Kailh hotswap MX socket, SW7 Kailh hotswap MX socket, SW8 Kailh hotswap MX socket, SW9 Kailh hotswap MX socket, U1 ProMicro, U2 SRV05-4

Commit message: Lotus 58 Classic
Tweaks

Signed-off-by: Markus Knutsson <markus.knutsson@tweety.se>
Parts:
- removed Logo1, Logo4: QMK_Logo, Logotypes:Powered_by_QMK
- added Logo5: QMK_Logo, Logotypes:qmk logo, B.Cu at (133.6, 113.1)
- added Logo6: QMK_Logo, Logotypes:qmk logo, F.Cu at (133.4, 113.1)
