File: Lotus 58 EZ/v1.00/Lotus58_EZ_100.kicad_pcb (KiCad board)
At the start: 2 copper layers, 139.1 x 107.7 mm, 158 parts, among them J1 USB_C_Receptacle_USB2.0, J3 USB_C_Receptacle_USB2.0, P1 OLED, Q1 2n2007, Q2 2n2007, Q3 2n2007, SW1 Kailh hotswap MX socket, SW10 Kailh hotswap MX socket, SW11 Kailh hotswap MX socket, SW12 Kailh hotswap MX socket, SW13 Kailh hotswap MX socket, SW14 Kailh hotswap MX socket, SW15 Kailh hotswap MX socket, SW16 Kailh hotswap MX socket, SW17 Kailh hotswap MX socket, SW18 Kailh hotswap MX socket, SW19 Kailh hotswap MX socket, SW2 Kailh hotswap MX socket, SW20 Kailh hotswap MX socket, SW21 Kailh hotswap MX socket, SW22 Kailh hotswap MX socket, SW23 Kailh hotswap MX socket, SW24 Kailh hotswap MX socket, SW25 Kailh hotswap MX socket, SW26 Kailh hotswap MX socket, SW27 Kailh hotswap MX socket, SW28 Kailh hotswap MX socket, SW29 Kailh hotswap MX socket, SW3 Kailh hotswap MX socket, SW30 Rotary_Encoder_Switch, SW31 Rotary_Encoder_Switch, SW4 Kailh hotswap MX socket, SW5 Kailh hotswap MX socket, SW6 Kailh hotswap MX socket, SW7 Kailh hotswap MX socket, SW8 Kailh hotswap MX socket, SW9 Kailh hotswap MX socket, U1 SRV05-4, U2 SRV05-4, U3 W25Q32JVUUIQ, U4 RP2040, U5 SPX3819M5-L-3-3/TR, U6 SN74LV1T34DBV, Y1 TXM12M0004252LBCEO00T

Commit message: Lotus 58 EZ
Tweaks

Signed-off-by: Markus Knutsson <markus.knutsson@tweety.se>
Parts:
- removed Q1, Q2, Q3: 2n2007, Package_TO_SOT_SMD:SOT-23
- moved U6 4.26 mm to (105.4, 55.1), turned to 0 degrees
- moved LED30 1.50 mm to (123.9, 51.0), turned to 90 degrees
- moved LED31 1.50 mm to (162.0, 50.9), turned to 90 degrees
- moved LED32 1.50 mm to (200.1, 55.4), turned to 90 degrees
- moved D6 0.95 mm to (200.4, 48.2)
- turned LED33 to 90 degrees
- turned LED34 to 90 degrees
- turned LED35 to 90 degrees
Connections:
- LED1 pad 3: Net-(LED1-GND) -> GND
- LED10 pad 3: Net-(LED1-GND) -> GND
- LED11 pad 3: Net-(LED1-GND) -> GND
- LED12 pad 3: Net-(LED1-GND) -> GND
- LED13 pad 3: Net-(LED1-GND) -> GND
- LED14 pad 3: Net-(LED1-GND) -> GND
- LED15 pad 3: Net-(LED1-GND) -> GND
- LED16 pad 3: Net-(LED1-GND) -> GND
- LED17 pad 3: Net-(LED1-GND) -> GND
- LED18 pad 3: Net-(LED1-GND) -> GND
- LED19 pad 3: Net-(LED1-GND) -> GND
- LED2 pad 3: Net-(LED1-GND) -> GND
- LED20 pad 3: Net-(LED1-GND) -> GND
- LED21 pad 3: Net-(LED1-GND) -> GND
- LED22 pad 3: Net-(LED1-GND) -> GND
- LED23 pad 3: Net-(LED1-GND) -> GND
- LED24 pad 3: Net-(LED1-GND) -> GND
- LED25 pad 3: Net-(LED1-GND) -> GND
- LED26 pad 3: Net-(LED1-GND) -> GND
- LED27 pad 3: Net-(LED1-GND) -> GND
- LED28 pad 3: Net-(LED1-GND) -> GND
- LED29 pad 2: unconnected-(LED29-DOUT-Pad2) -> RGB_LINK
- LED29 pad 3: Net-(LED1-GND) -> GND
- LED3 pad 3: Net-(LED1-GND) -> GND
- LED30 pad 3: Net-(LED30-GND) -> GND
- LED30 pad 4: RGB_5 -> RGB_LINK
- LED31 pad 3: Net-(LED30-GND) -> GND
- LED32 pad 3: Net-(LED30-GND) -> GND
- LED33 pad 3: Net-(LED30-GND) -> GND
- LED34 pad 3: Net-(LED30-GND) -> GND
- LED35 pad 3: Net-(LED30-GND) -> GND
- LED4 pad 3: Net-(LED1-GND) -> GND
- LED5 pad 3: Net-(LED1-GND) -> GND
- LED6 pad 3: Net-(LED1-GND) -> GND
- LED7 pad 3: Net-(LED1-GND) -> GND
- LED8 pad 3: Net-(LED1-GND) -> GND
- LED9 pad 3: Net-(LED1-GND) -> GND
- U4 pad 40: GLOW -> unconnected-(U4-GPIO28_ADC2-Pad40)
- U4 pad 41: KEY -> unconnected-(U4-GPIO29_ADC3-Pad41)
Routing:
- net Net-(LED1-GND): track 689.1 -> 0.00 mm, vias 29 -> 0
- net Net-(LED30-GND): track 296.4 -> 0.00 mm, vias 15 -> 0
- net RGB_LINK: track 0.00 -> 115.7 mm, vias 0 -> 3
- net GND: track 24.4 -> 139.1 mm, vias 34 -> 70
- net GLOW: track 31.1 -> 0.00 mm
- net KEY: track 26.7 -> 0.00 mm, vias 3 -> 0
- net RGB_5: track 23.7 -> 8.06 mm, vias 2 -> 1
- net Net-(LED32-DOUT): track 67.2 -> 59.6 mm
- net RGB: track 20.3 -> 26.2 mm
- net Net-(LED28-DOUT): track 19.6 -> 22.4 mm
- net Net-(LED31-DOUT): track 43.6 -> 46.2 mm, vias 3 -> 2
- net row0: track 140.0 -> 137.5 mm
- net +5V: track 785.0 -> 782.6 mm, vias 49 -> 48
- net Net-(LED33-DOUT): track 60.8 -> 58.8 mm, vias 3 -> 2
- net Net-(LED34-DOUT): track 72.0 -> 73.9 mm, vias 3 -> 5
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Other:
- board text added: "For basic core functionality, the hot-swap sockets needs to be added to the REAR FACE for each hand, and the jumper assigning hands needs to be closed."
- board text added: "Place reset switch on PCB REAR FACE"
- board text added: "The reset switch is soldered to the REAR FACE of the PCB, matching case designs. Encoder and/or OLED is soldered to the FRONT FACE of the PCB."
- board text added: "This design intended for use with SK6803 mini-E RGB ONLY! Place Per-Key RGB's on REAR FACE & Glow RGB on FRONT FACE of the PCB, facing down and align marked leg."
- board text removed: "For basic core functionality, the hot-swap sockets needs to be added to the REAR FACE for each hand, and the jumper to assign hands needs to be closed."
- board text removed: "Place Per-Key RGB on REAR FACE of PCB, facing down and align marked leg. Place Glow RGB on FRONT FACE of PCB, facing down and align marked leg."
- board text removed: "Place switches on PCB REAR FACE"
- board text removed: "The reset switch and RGB selector switch is soldered to the REAR FACE of the PCB, to match the 3D printed case. Encoder or OLED is soldered to the FRONT FACE of the PCB."
