File: Lotus 58 EZ/v1.00/Lotus58_EZ_100.kicad_sch (KiCad schematic)
At the start: 158 parts, among them J1 USB_C_Receptacle_USB2.0, J3 USB_C_Receptacle_USB2.0, P1 OLED, Q1 2n2007, Q2 2n2007, Q3 2n2007, SW1 Kailh hotswap MX socket, SW10 Kailh hotswap MX socket, SW11 Kailh hotswap MX socket, SW12 Kailh hotswap MX socket, SW13 Kailh hotswap MX socket, SW14 Kailh hotswap MX socket, SW15 Kailh hotswap MX socket, SW16 Kailh hotswap MX socket, SW17 Kailh hotswap MX socket, SW18 Kailh hotswap MX socket, SW19 Kailh hotswap MX socket, SW2 Kailh hotswap MX socket, SW20 Kailh hotswap MX socket, SW21 Kailh hotswap MX socket, SW22 Kailh hotswap MX socket, SW23 Kailh hotswap MX socket, SW24 Kailh hotswap MX socket, SW25 Kailh hotswap MX socket, SW26 Kailh hotswap MX socket, SW27 Kailh hotswap MX socket, SW28 Kailh hotswap MX socket, SW29 Kailh hotswap MX socket, SW3 Kailh hotswap MX socket, SW30 Rotary_Encoder_Switch, SW31 Rotary_Encoder_Switch, SW4 Kailh hotswap MX socket, SW5 Kailh hotswap MX socket, SW6 Kailh hotswap MX socket, SW7 Kailh hotswap MX socket, SW8 Kailh hotswap MX socket, SW9 Kailh hotswap MX socket, U1 SRV05-4, U2 SRV05-4, U3 W25Q32JVUUIQ, U4 RP2040, U5 SPX3819M5-L-3-3/TR, U6 SN74LV1T34DBV, Y1 TXM12M0004252LBCEO00T

Commit message: Lotus 58 EZ
Tweaks

Signed-off-by: Markus Knutsson <markus.knutsson@tweety.se>
Parts:
- removed Q1, Q2, Q3: 2n2007, Package_TO_SOT_SMD:SOT-23, symbol Device:Q_NMOS_GSD
Connections:
- net GND: now also LED1.3 (GND), LED10.3 (GND), LED11.3 (GND), LED12.3 (GND), LED13.3 (GND), LED14.3 (GND), LED15.3 (GND), LED16.3 (GND), LED17.3 (GND), LED18.3 (GND), LED19.3 (GND), LED2.3 (GND), LED20.3 (GND), LED21.3 (GND), LED22.3 (GND), LED23.3 (GND), LED24.3 (GND), LED25.3 (GND), LED26.3 (GND), LED27.3 (GND), LED28.3 (GND), LED29.3 (GND), LED3.3 (GND), LED30.3 (GND), LED31.3 (GND), LED32.3 (GND), LED33.3 (GND), LED34.3 (GND), LED35.3 (GND), LED4.3 (GND), LED5.3 (GND), LED6.3 (GND), LED7.3 (GND), LED8.3 (GND), LED9.3 (GND)
- net RGB_5: no longer LED30.4 (DIN)
- net RGB_LINK: now reaches LED29.2 (DOUT)
- net RGB_LINK: now also LED30.4 (DIN)
- net GLOW: no longer names the net of U4.40 (GPIO28_ADC2)
- net KEY: no longer names the net of U4.41 (GPIO29_ADC3)
- no-connect marks 21 -> 22
Other:
- moved on the sheet: C1, C2, FB1, FB4, J3, LED1, LED10, LED11, LED12, LED13, LED14, LED15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
