File: Lotus 58 TRRS/v1.30/Lotus58_Glow_130.kicad_pcb (KiCad board)
At the start: 2 copper layers, 139.1 x 107.7 mm, 116 parts, among them J1 PJ-320A, J2 Conn_01x02, P1 OLED, SW1 Kailh hotswap MX socket, SW10 Kailh hotswap MX socket, SW11 Kailh hotswap MX socket, SW12 Kailh hotswap MX socket, SW13 Kailh hotswap MX socket, SW14 Kailh hotswap MX socket, SW15 Kailh hotswap MX socket, SW16 Kailh hotswap MX socket, SW17 Kailh hotswap MX socket, SW18 Kailh hotswap MX socket, SW19 Kailh hotswap MX socket, SW2 Kailh hotswap MX socket, SW20 Kailh hotswap MX socket, SW21 Kailh hotswap MX socket, SW22 Kailh hotswap MX socket, SW23 Kailh hotswap MX socket, SW24 Kailh hotswap MX socket, SW25 Kailh hotswap MX socket, SW26 Kailh hotswap MX socket, SW27 Kailh hotswap MX socket, SW28 Kailh hotswap MX socket, SW29 Kailh hotswap MX socket, SW3 Kailh hotswap MX socket, SW30 Rotary_Encoder_Switch, SW31 Rotary_Encoder_Switch, SW4 Kailh hotswap MX socket, SW5 Kailh hotswap MX socket, SW6 Kailh hotswap MX socket, SW7 Kailh hotswap MX socket, SW8 Kailh hotswap MX socket, SW9 Kailh hotswap MX socket, U1 ProMicro, U2 SRV05-4

Commit message: Lotus 58 - TRRS Link v1.30
release ready

Signed-off-by: Markus Knutsson <markus.knutsson@tweety.se>
Parts:
- removed the Logo2 at (103.2, 117.2)
- added G***: LOGO, Logotypes:RoHs, F.Cu at (154.2, 112.3)
- added G***: LOGO, Logotypes:RoHs, B.Cu at (160.0, 112.3)
- added Logo5: CE_Logo, Logotypes:CE, F.Cu at (161.1, 112.3)
- added Logo6: CE_Logo, Logotypes:CE, B.Cu at (153.3, 112.3)
- added Logo7: CC-BY-SA-4.0, Logotypes:CC_BY_SA_40_line, F.Cu at (135.8, 113.4)
- added Logo8: QMK_Logo, Logotypes:qmk logo, F.Cu at (183.0, 118.6)
- C1, C2: value 100nF -> 50V/100nF axial
- LED10, LED11, LED12, LED13, LED14, LED15, LED16, LED17, LED18, LED19, LED20, LED21, LED22, LED23, LED24, LED25, LED26, LED27, LED28, LED29, LED30, LED31, LED32, LED33, LED34, LED35, LED7, LED8, LED9: value SK6812MINI-E -> SK6803MINI-E
- Logo2: moved to B.Cu
- SW30, SW31: value Rotary_Encoder_Switch -> EC_11
- U1: value ProMicro -> Controller; footprint Keyboard Controllers:ProMicro_Reversible_mod -> Keyboard Controllers:ProMicro_Reversible_orig
- moved Logo1 31.0 mm to (183.2, 118.6)
- moved Logo2 15.4 mm to (135.8, 113.4), turned to 180 degrees
- moved C1 0.12 mm to (104.9, 53.4), turned to 135 degrees
Connections:
- C1 pad 1: B -> GND
- C1 pad 2: GND -> B
- S1 pad NO: Net-(S1-PadNO) -> unconnected-(S1-PadNO)
- S2 pad NO: Net-(S1-PadNO) -> unconnected-(S1-PadNO)
Routing:
- net unconnected-(S1-PadNO): track 0.00 -> 6.72 mm, vias 0 -> 1
- net Net-(S1-PadNO): track 6.72 -> 0.00 mm, vias 1 -> 0
Other:
- board text added: "Markus Knutsson 2025 https://github.com/TweetyDaBird"
- board text removed: "Markus Knutsson - 2024 https://github.com/TweetyDaBird"
