File: Lotus 58 TRRS/v1.30/Lotus58_Glow_130.kicad_sch (KiCad schematic)
At the start: 115 parts, among them J1 PJ-320A, J2 Conn_01x02, P1 OLED, SW1 Kailh hotswap MX socket, SW10 Kailh hotswap MX socket, SW11 Kailh hotswap MX socket, SW12 Kailh hotswap MX socket, SW13 Kailh hotswap MX socket, SW14 Kailh hotswap MX socket, SW15 Kailh hotswap MX socket, SW16 Kailh hotswap MX socket, SW17 Kailh hotswap MX socket, SW18 Kailh hotswap MX socket, SW19 Kailh hotswap MX socket, SW2 Kailh hotswap MX socket, SW20 Kailh hotswap MX socket, SW21 Kailh hotswap MX socket, SW22 Kailh hotswap MX socket, SW23 Kailh hotswap MX socket, SW24 Kailh hotswap MX socket, SW25 Kailh hotswap MX socket, SW26 Kailh hotswap MX socket, SW27 Kailh hotswap MX socket, SW28 Kailh hotswap MX socket, SW29 Kailh hotswap MX socket, SW3 Kailh hotswap MX socket, SW30 Rotary_Encoder_Switch, SW31 Rotary_Encoder_Switch, SW4 Kailh hotswap MX socket, SW5 Kailh hotswap MX socket, SW6 Kailh hotswap MX socket, SW7 Kailh hotswap MX socket, SW8 Kailh hotswap MX socket, SW9 Kailh hotswap MX socket, U1 ProMicro, U2 SRV05-4

Commit message: Lotus 58 - TRRS Link v1.30
Signed-off-by: Markus Knutsson <markus.knutsson@tweety.se>
Parts:
- added JP2: LEFT, Keyboard Common:Jumper_min_v2, symbol Device:Jumper_NO_Small
- added JP3: RIGHT, Keyboard Common:Jumper_min_v2, symbol Device:Jumper_NO_Small
- LED1, LED2, LED3, LED4, LED5, LED6: footprint Keyboard RGB:MX_SK6812MINI-E_REVERSIBLE_special_v2 -> Keyboard RGB:MX_SK6812MINI-E_REVERSIBLE
- U1: footprint Keyboard Controllers:ProMicro_Reversible_mod -> Keyboard Controllers:ProMicro_Reversible_orig; symbol Keyboard_Controllers:ProMicro_jumpers_v2 -> keebio:ProMicro
Connections:
- net GND: now also JP3.1; no longer U1.12B
- net VCC: now also JP2.1; no longer U1.12A (9/PB5)
- new net Hand: JP2.2, JP3.2, U1.12 (9/PB5)
- no-connect marks 5 -> 6

Commit message: Lotus 58 - TRRS Link v1.30
release ready

Signed-off-by: Markus Knutsson <markus.knutsson@tweety.se>
Parts:
- removed JP2: LEFT, Keyboard Common:Jumper_min_v2, symbol Device:Jumper_NO_Small
- removed JP3: RIGHT, Keyboard Common:Jumper_min_v2, symbol Device:Jumper_NO_Small
- added Logo10, Logo3, Logo4, Logo9: RoHS_Logo, Logotypes:RoHS, symbol Logotypes:RoHS_Logo
- added Logo5, Logo6: CE_Logo, Logotypes:CE, symbol Logotypes:CE_Logo
- added Logo7: CC-BY-SA-4.0, Logotypes:CC_BY_SA_40_line, symbol Logotypes:CC-BY-SA-4.0
- added Logo8: QMK_Logo, Logotypes:qmk logo, symbol Logotypes:QMK_Logo
- C1, C2: value 100nF -> 50V/100nF axial
- J2, JP5, TH1, TH2, TH3, TH4, TH5: now left out of the parts list
- LED1, LED10, LED11, LED12, LED13, LED14, LED15, LED16, LED17, LED18, LED19, LED2, LED20, LED21, LED22, LED23, LED24, LED25, LED26, LED27, LED28, LED29, LED3, LED30, LED31, LED32, LED33, LED34, LED35, LED4, LED5, LED6, LED7, LED8, LED9: value SK6812MINI-E -> SK6803MINI-E
- SW30, SW31: value Rotary_Encoder_Switch -> EC_11
- U1: value ProMicro -> Controller
Other:
- title: Lotus 58 Glow -> Lotus 58 - TRRS Link
