File: Lotus 58 USB-C/v1.51/Lotus58_Glow_151.kicad_pcb (KiCad board)
At the start: 2 copper layers, 139.1 x 107.7 mm, 151 parts, among them J1 USB_C_Receptacle_USB2.0, P1 OLED, SW1 Kailh hotswap MX socket, SW10 Kailh hotswap MX socket, SW11 Kailh hotswap MX socket, SW12 Kailh hotswap MX socket, SW13 Kailh hotswap MX socket, SW14 Kailh hotswap MX socket, SW15 Kailh hotswap MX socket, SW16 Kailh hotswap MX socket, SW17 Kailh hotswap MX socket, SW18 Kailh hotswap MX socket, SW19 Kailh hotswap MX socket, SW2 Kailh hotswap MX socket, SW20 Kailh hotswap MX socket, SW21 Kailh hotswap MX socket, SW22 Kailh hotswap MX socket, SW23 Kailh hotswap MX socket, SW24 Kailh hotswap MX socket, SW25 Kailh hotswap MX socket, SW26 Kailh hotswap MX socket, SW27 Kailh hotswap MX socket, SW28 Kailh hotswap MX socket, SW29 Kailh hotswap MX socket, SW3 Kailh hotswap MX socket, SW4 Kailh hotswap MX socket, SW5 Kailh hotswap MX socket, SW6 Kailh hotswap MX socket, SW7 Kailh hotswap MX socket, SW8 Kailh hotswap MX socket, SW9 Kailh hotswap MX socket, U1 ProMicro, U2 SRV05-4, U3 SRV05-4

Commit message: Lotus 58 - TRRS Link v1.30
release ready

Signed-off-by: Markus Knutsson <markus.knutsson@tweety.se>
Parts:
- added Logo7: CC-BY-SA-4.0, Logotypes:CC_BY_SA_40_line, B.Cu at (136.3, 113.6)
- added Logo8: CC-BY-SA-4.0, Logotypes:CC_BY_SA_40_line, F.Cu at (135.8, 113.6)
- C1, C2: value 100nF -> 50V/100nF axial
- ENC30, ENC31: value Rotary_Encoder_Click -> EC11
- FB1, FB2, FB3, FB4: value Ferrite Bead -> 0603/150-200R
- J1: value USB_C_Receptacle_USB2.0 -> HRO-TYPE-C-31-M-13x
- U1: value ProMicro -> Controller
- moved Logo1 49.5 mm to (181.8, 118.5)
- moved Logo2 49.5 mm to (181.9, 118.5)
- moved Logo6 2.64 mm to (154.1, 112.3)
- moved G*** 2.64 mm to (154.1, 112.3)
- moved G*** 1.14 mm to (160.7, 112.3)
- moved Logo4 1.14 mm to (160.7, 112.3)
Other:
- board text added: "Markus Knutsson 2025 https://github.com/TweetyDaBird"
- board text added: "USB-C link v1.5.1"
- board text removed: "Markus Knutsson 2024 https://github.com/TweetyDaBird Licensed under CERN-OHL-S v2+"
- board text removed: "USB-C link v1.5.0"
