File: Lotus 58 USB-C/v1.51/Lotus58_Glow_151.kicad_sch (KiCad schematic)
At the start: 152 parts, among them J1 USB_C_Receptacle_USB2.0, P1 OLED, SW1 Kailh hotswap MX socket, SW10 Kailh hotswap MX socket, SW11 Kailh hotswap MX socket, SW12 Kailh hotswap MX socket, SW13 Kailh hotswap MX socket, SW14 Kailh hotswap MX socket, SW15 Kailh hotswap MX socket, SW16 Kailh hotswap MX socket, SW17 Kailh hotswap MX socket, SW18 Kailh hotswap MX socket, SW19 Kailh hotswap MX socket, SW2 Kailh hotswap MX socket, SW20 Kailh hotswap MX socket, SW21 Kailh hotswap MX socket, SW22 Kailh hotswap MX socket, SW23 Kailh hotswap MX socket, SW24 Kailh hotswap MX socket, SW25 Kailh hotswap MX socket, SW26 Kailh hotswap MX socket, SW27 Kailh hotswap MX socket, SW28 Kailh hotswap MX socket, SW29 Kailh hotswap MX socket, SW3 Kailh hotswap MX socket, SW30 Rotary_Encoder_Switch, SW31 Rotary_Encoder_Switch, SW32 MSK12C02, SW33 MSK12C02, SW4 Kailh hotswap MX socket, SW5 Kailh hotswap MX socket, SW6 Kailh hotswap MX socket, SW7 Kailh hotswap MX socket, SW8 Kailh hotswap MX socket, SW9 Kailh hotswap MX socket, U1 ProMicro, U2 SRV05-4, U3 SRV05-4

Commit message: Lotus 58 - USB Link v1.51
adjusted RGB Gl
ow, Silkscreen

Signed-off-by: Markus Knutsson <markus.knutsson@tweety.se>
Parts:
- removed JP2, JP3: LEFT, Keyboard Common:Jumper_min_v2, symbol Jumper:Jumper_2_Open
- removed JP4: RIGHT, Keyboard Common:Jumper_min_v2, symbol Jumper:Jumper_2_Open
- removed SW25: Kailh hotswap MX socket, Keyboard Switches:SW_MX_HotSwap_Reversible_FOR encoder, symbol Keyboard Switches:SW_Push_GND
- removed SW32, SW33: MSK12C02, Keyboard Common:MSK12C02, symbol Keyboard Common:MSK12C02
- added Logo3, Logo5: RoHS_Logo, Logotypes:RoHS, symbol Logotypes:RoHS_Logo
- added Logo4, Logo6: CE_Logo, Logotypes:CE, symbol Logotypes:CE_Logo
- added SW25: Kailh hotswap MX socket, Keyboard Switches:SW_MX_HotSwap_Reversible, symbol Switch:SW_Push
- ENC30: renamed from SW30; value Rotary_Encoder_Switch -> Rotary_Encoder_Click
- ENC31: renamed from SW31; value Rotary_Encoder_Switch -> Rotary_Encoder_Click; footprint Keyboard Encoders:Encoder_Alps_EC11E_Small -> Keyboard Encoders:Encoder_Alps_EC11E_Small_onkey
- LED30, LED31, LED32, LED33, LED34, LED35: value SK6812MINI-E -> SK6803MINI-E; footprint Keyboard RGB:MX_SK6812MINI-E_REVERSIBLE -> Keyboard RGB:MX_SK6812MINI-E_REVERSIBLE_special_v2
- Logo2: footprint Logotypes:qmk logo -> Logotypes:RoHS
- U1: footprint Keyboard Controllers:ProMicro_jumpers_V2 -> Keyboard Controllers:ProMicro_jumpers_V3
Connections:
- net PWR_KEY is gone; now on net VCC: LED1.1 (VDD), LED10.1 (VDD), LED11.1 (VDD), LED12.1 (VDD), LED13.1 (VDD), LED14.1 (VDD), LED15.1 (VDD), LED16.1 (VDD), LED17.1 (VDD), LED18.1 (VDD), LED19.1 (VDD), LED2.1 (VDD), LED20.1 (VDD), LED21.1 (VDD), LED22.1 (VDD), LED23.1 (VDD), LED24.1 (VDD), LED25.1 (VDD), LED26.1 (VDD), LED27.1 (VDD), LED28.1 (VDD), LED29.1 (VDD), LED3.1 (VDD), LED4.1 (VDD), LED5.1 (VDD), LED6.1 (VDD), LED7.1 (VDD), LED8.1 (VDD), LED9.1 (VDD)
- net Alt: now also SW25.1
- net GND: now also ENC30.MP (GND), ENC31.MP (GND), U1.12B; no longer ENC30.MP1 (GND), ENC30.MP2 (GND), ENC31.MP1 (GND), ENC31.MP2 (GND)
- net LED: now also JP1.2 (B); no longer LED1.4 (DIN)
- net VCC: now also LED30.1 (VDD), LED31.1 (VDD), LED32.1 (VDD), LED33.1 (VDD), LED34.1 (VDD), LED35.1 (VDD), U1.12A (9/PB5); no longer JP1.2 (B)
- net col5: now also SW25.2
- net at U1.E (0), U1.F (0), U1.G (0)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: no longer U1.A (0), U1.B (0), U1.C (0), U1.D (0)
- net KEY: now reaches LED35.2 (DOUT)
- net KEY: now also JP1.1 (A), LED1.4 (DIN)
- removed net Hand: U1.12 (9/PB5)
- removed net PWR_GLOW: JP1.1 (A), LED30.1 (VDD), LED31.1 (VDD), LED32.1 (VDD), LED33.1 (VDD), LED34.1 (VDD), LED35.1 (VDD)
- new net: U1.C (0), U1.D (0)
- no-connect marks 11 -> 10
Other:
- note removed: "VCC/High = Left GND/Low = Right"
- title: Lotus 58 Glow -> Lotus 58 - USB Link
- moved on the sheet: C1, C2, D1, D10, D11, D12, D13, D14, D15, D16, D17, D18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

Commit message: Corrected iBom
USB v1.51

Signed-off-by: Markus Knutsson <markus.knutsson@tweety.se>
Parts:
- C1, C2: value 100nF -> 50V/100nF axial; now fitted
- ENC30, ENC31: value Rotary_Encoder_Click -> EC11
- FB1, FB2, FB3, FB4: value Ferrite Bead -> 0603/150-200R
- J1: value USB_C_Receptacle_USB2.0 -> HRO-TYPE-C-31-M-13x
- JP1, TH1, TH2, TH3, TH4, TH5: now left out of the parts list
- U1: value ProMicro -> Controller
Other:
- moved on the sheet: Logo2
Changed lines of the file:
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@@
 			)
 		)
-		(property "Value" "ProMicro"
+		(property "Value" "Controller"
 			(at 336.55 95.25 0)
 			(effects
@@
 		(unit 1)
 		(exclude_from_sim no)
-		(in_bom yes)
+		(in_bom no)
 		(on_board yes)
 		(dnp yes)
@@
 		(unit 1)
 		(exclude_from_sim no)
-		(in_bom yes)
+		(in_bom no)
 		(on_board yes)
 		(dnp yes)
@@
 		(unit 1)
 		(exclude_from_sim no)
-		(in_bom yes)
+		(in_bom no)
 		(on_board yes)
 		(dnp yes)
@@
 		(unit 1)
 		(exclude_from_sim no)
-		(in_bom yes)
+		(in_bom no)
 		(on_board yes)
 		(dnp yes)
@@
 		(unit 1)
 		(exclude_from_sim no)
-		(in_bom yes)
+		(in_bom no)
 		(on_board yes)
 		(dnp yes)
@@
 			)
 		)
-		(property "Value" "Rotary_Encoder_Click"
+		(property "Value" "EC11"
 			(at 175.26 97.79 0)
 			(effects
@@
 		(in_bom yes)
 		(on_board yes)
-		(dnp yes)
+		(dnp no)
 		(property "Reference" "C1"
 			(at 207.2132 106.5784 0)
@@
 			)
 		)
-		(property "Value" "100nF"
+		(property "Value" "50V/100nF axial"
 			(at 207.2132 104.267 0)
 			(effects
@@
 		(in_bom yes)
 		(on_board yes)
-		(dnp yes)
+		(dnp no)
 		(property "Reference" "C2"
 			(at 211.8868 109.3216 0)
@@
 			)
 		)
-		(property "Value" "100nF"
+		(property "Value" "50V/100nF axial"
 			(at 211.8868 111.633 0)
 			(effects
@@
 			)
 		)
-		(property "Value" "Rotary_Encoder_Click"
+		(property "Value" "EC11"
 			(at 228.6 43.18 0)
 			(effects
@@
 			)
 		)
-		(property "Value" "Ferrite Bead"
+		(property "Value" "0603/150-200R"
 			(at 185.3819 243.078 90)
 			(effects
@@
 	(symbol
 		(lib_id "Logotypes:RoHS_Logo")
-		(at 184.15 283.21 0)
+		(at 176.53 271.78 0)
 		(unit 1)
 		(exclude_from_sim no)
@@
 		(fields_autoplaced yes)
 		(property "Reference" "Logo3"
-			(at 184.15 273.685 0)
+			(at 176.53 262.255 0)
 			(effects
 				(font
@@
 		)
 		(property "Value" "RoHS_Logo"
-			(at 191.77 281.9399 0)
+			(at 184.15 270.5099 0)
 			(effects
 				(font
@@
 		)
 		(property "Footprint" "Logotypes:RoHS"
-			(at 184.15 283.21 0)
+			(at 176.53 271.78 0)
 			(effects
 				(font
@@
 		)
 		(property "Datasheet" ""
-			(at 184.15 283.21 0)
+			(at 176.53 271.78 0)
 			(effects
 				(font
@@
 		)
 		(property "Description" ""
-			(at 184.15 283.21 0)
+			(at 176.53 271.78 0)
 			(effects
 				(font
@@
 			)
 		)
-		(property "Value" "USB_C_Receptacle_USB2.0"
+		(property "Value" "HRO-TYPE-C-31-M-13x"
 			(at 189.23 198.882 0)
 			(effects
@@
 		(unit 1)
 		(exclude_from_sim no)
-		(in_bom yes)
+		(in_bom no)
 		(on_board yes)
 		(dnp yes)
@@
 	(symbol
 		(lib_id "Logotypes:CE_Logo")
-		(at 184.15 289.56 0)
+		(at 176.53 278.13 0)
 		(unit 1)
 		(exclude_from_sim no)
@@
 		(fields_autoplaced yes)
 		(property "Reference" "Logo6"
-			(at 184.15 280.035 0)
+			(at 176.53 268.605 0)
 			(effects
 				(font
@@
 		)
 		(property "Value" "CE_Logo"
-			(at 191.77 288.2899 0)
+			(at 184.15 276.8599 0)
 			(effects
 				(font
@@
 		)
 		(property "Footprint" "Logotypes:CE"
-			(at 184.15 289.56 0)
+			(at 176.53 278.13 0)
 			(effects
 				(font
@@
 		)
 		(property "Datasheet" ""
-			(at 184.15 289.56 0)
+			(at 176.53 278.13 0)
 			(effects
 				(font
@@
 		)
 		(property "Description" ""
-			(at 184.15 289.56 0)
+			(at 176.53 278.13 0)
 			(effects
 				(font
@@
 	(symbol
 		(lib_id "Logotypes:QMK_Logo")
-		(at 207.01 276.86 0)
+		(at 201.93 265.43 0)
 		(unit 1)
 		(exclude_from_sim no)
@@
 		(fields_autoplaced yes)
 		(property "Reference" "Logo2"
-			(at 207.01 267.335 0)
+			(at 201.93 255.905 0)
 			(effects
 				(font
@@
 		)
 		(property "Value" "QMK_Logo"
-			(at 207.01 269.875 0)
+			(at 201.93 258.445 0)
 			(effects
 				(font
@@
 		)
 		(property "Footprint" "Logotypes:RoHS"
-			(at 207.01 276.86 0)
+			(at 201.93 265.43 0)
 			(effects
 				(font
@@
 		)
 		(property "Datasheet" ""
-			(at 207.01 276.86 0)
+			(at 201.93 265.43 0)
 			(effects
 				(font
@@
 		)
 		(property "Description" ""
-			(at 207.01 276.86 0)
+			(at 201.93 265.43 0)
 			(effects
 				(font
@@
 	(symbol
 		(lib_id "Logotypes:RoHS_Logo")
-		(at 209.55 289.56 0)
+		(at 201.93 278.13 0)
 		(unit 1)
 		(exclude_from_sim no)
@@
 		(fields_autoplaced yes)
 		(property "Reference" "Logo5"
-			(at 209.55 280.035 0)
+			(at 201.93 268.605 0)
 			(effects
 				(font
@@
 		)
 		(property "Value" "RoHS_Logo"
-			(at 217.17 288.2899 0)
+			(at 209.55 276.8599 0)
 			(effects
 				(font
@@
 		)
 		(property "Footprint" "Logotypes:RoHS"
-			(at 209.55 289.56 0)
+			(at 201.93 278.13 0)
 			(effects
 				(font
@@
 		)
 		(property "Datasheet" ""
-			(at 209.55 289.56 0)
+			(at 201.93 278.13 0)
 			(effects
 				(font
@@
 		)
 		(property "Description" ""
-			(at 209.55 289.56 0)
+			(at 201.93 278.13 0)
 			(effects
 				(font
@@
 			)
 		)
-		(property "Value" "Ferrite Bead"
+		(property "Value" "0603/150-200R"
 			(at 217.1319 199.898 90)
 			(effects
@@
 			)
 		)
-		(property "Value" "Ferrite Bead"
+		(property "Value" "0603/150-200R"
 			(at 185.3819 243.078 90)
 			(effects
@@
 	(symbol
 		(lib_id "Logotypes:CE_Logo")
-		(at 209.55 281.94 0)
+		(at 201.93 271.78 0)
 		(unit 1)
 		(exclude_from_sim no)
@@
 		(fields_autoplaced yes)
 		(property "Reference" "Logo4"
-			(at 209.55 272.415 0)
+			(at 201.93 262.255 0)
 			(effects
 				(font
@@
 		)
 		(property "Value" "CE_Logo"
-			(at 217.17 280.6699 0)
+			(at 209.55 270.5099 0)
 			(effects
 				(font
@@
 		)
 		(property "Footprint" "Logotypes:CE"
-			(at 209.55 281.94 0)
+			(at 201.93 271.78 0)
 			(effects
 				(font
@@
 		)
 		(property "Datasheet" ""
-			(at 209.55 281.94 0)
+			(at 201.93 271.78 0)
 			(effects
 				(font
@@
 		)
 		(property "Description" ""
-			(at 209.55 281.94 0)
+			(at 201.93 271.78 0)
 			(effects
 				(font
@@
 			)
 		)
-		(property "Value" "Ferrite Bead"
+		(property "Value" "0603/150-200R"
 			(at 217.1319 199.898 90)
 			(effects
@@
 		(lib_name "QMK_Logo_1")
 		(lib_id "Logotypes:QMK_Logo")
-		(at 184.15 276.86 0)
+		(at 176.53 265.43 0)
 		(unit 1)
 		(exclude_from_sim no)
@@
 		(fields_autoplaced yes)
 		(property "Reference" "Logo1"
-			(at 184.15 267.335 0)
+			(at 176.53 255.905 0)
 			(effects
 				(font
@@
 		)
 		(property "Value" "QMK_Logo"
-			(at 184.404 271.526 0)
+			(at 176.784 260.096 0)
 			(effects
 				(font
@@
 		)
 		(property "Footprint" "Logotypes:qmk logo"
-			(at 184.15 276.86 0)
+			(at 176.53 265.43 0)
 			(effects
 				(font
@@
 		)
 		(property "Datasheet" ""
-			(at 184.15 276.86 0)
+			(at 176.53 265.43 0)
 			(effects
 				(font
@@
 		)
 		(property "Description" ""
-			(at 184.15 276.86 0)
+			(at 176.53 265.43 0)
 			(effects
 				(font

Commit message: Lotus 58 - TRRS Link v1.30
release ready

Signed-off-by: Markus Knutsson <markus.knutsson@tweety.se>
Parts:
- added Logo7, Logo8: CC-BY-SA-4.0, Logotypes:CC_BY_SA_40_line, symbol Logotypes:CC-BY-SA-4.0
Other:
- moved on the sheet: FB1, FB2, FB3, FB4, J1, JP1, P1, U2, U3
